File: KanaType.kicad_pcb (KiCad board)
At the start: 2 copper layers, 84.8 x 57 mm, 61 parts, among them J1 Conn_01x04_Socket, SW1 SW_Push, SW10 SW_Push, SW11 SW_Push, SW12 SW_Push, SW13 SW_Push, SW14 SW_Push, SW15 SW_Push, SW16 SW_Push, SW17 SW_Push, SW18 SW_Push, SW19 SW_Push, SW2 SW_Push, SW20 SW_Push, SW21 SW_Push, SW22 SW_Push, SW23 SW_Push, SW24 SW_Push, SW25 SW_Push, SW26 SW_Push, SW27 SW_Push, SW28 SW_Push, SW29 SW_Push, SW3 SW_Push, SW30 SW_Push, SW31 SW_Push, SW32 SW_Push, SW33 SW_Push, SW34 SW_Push, SW35 SW_Push, SW36 SW_Push, SW37 SW_Push, SW38 SW_Push, SW39 SW_Push, SW4 SW_Push, SW40 SW_Push, SW41 SW_Push, SW42 SW_Push, SW43 SW_Push, SW44 SW_Push, SW45 SW_Push, SW46 SW_Push, SW47 SW_Push, SW48 SW_Push, SW49 SW_Push, SW5 SW_Push, SW51 SW_Push, SW53 SW_Push, SW55 SW_Push, SW57 SW_Push, SW59 SW_Push, SW6 SW_Push, SW61 SW_Push, SW63 SW_Push, SW7 SW_Push, SW8 SW_Push, SW9 SW_Push, U1 Adafruit-Feather-RP2040

Commit message: Hardware: E9 column pull-downs, OLED support parts, WAKE/RESET
- R1-R8: 8.2k pull-downs on COL1-COL8. Neutralize the RP2350-E9 erratum
  (whose internal pull-downs are unreliable) and hold the columns low when
  no key is pressed. This commits the board to ACTIVE-HIGH scanning
  permanently: columns_to_anodes=False everywhere, non-negotiable.
- R9, R10: 8.2k I2C pull-ups on SDA/SCL, so the bus is self-sufficient
  regardless of what an attached module provides.
- R11: 1k series for WAKE1, capping fault current at 3.3 mA when the key
  drives COL8 against its 8.2k pull-down.
- C1: 10 uF bulk cap across 3.3 V near J1, as the OLED transient reservoir.
- RESET1 / WAKE1 tactile switches.

Also corrects the matrix wiring: every switch now uses pad 2 -> row and
pad 4 -> column. The LCSC symbol shows diagonal internal pairing but the
YTS810SJK datasheet specifies edge pairing ({1,2} and {3,4}), and the
original pad-3 wiring shorted every key in the matrix. Caught before
fabrication.

DRC, ERC and schematic-parity were clean at the 2026-08 audit.

Co-Authored-By: Claude Opus 5 <noreply@anthropic.com>
Parts:
- added C1: 10 μF, Capacitor_SMD:C_0805_2012Metric_Pad1.18x1.45mm_HandSolder, F.Cu at (206.4, 40.0)
- added R1: 8.2k, Resistor_SMD:R_0805_2012Metric_Pad1.20x1.40mm_HandSolder, F.Cu at (191.0, 45.5)
- added R10: 8.2k, Resistor_SMD:R_0805_2012Metric_Pad1.20x1.40mm_HandSolder, F.Cu at (218.2, 39.5)
- added R11: 1k, Resistor_SMD:R_0805_2012Metric_Pad1.20x1.40mm_HandSolder, F.Cu at (158.2, 43.5)
- added R2: 8.2k, Resistor_SMD:R_0805_2012Metric_Pad1.20x1.40mm_HandSolder, F.Cu at (199.0, 48.5)
- added R3: 8.2k, Resistor_SMD:R_0805_2012Metric_Pad1.20x1.40mm_HandSolder, F.Cu at (187.0, 48.5)
- added R4: 8.2k, Resistor_SMD:R_0805_2012Metric_Pad1.20x1.40mm_HandSolder, F.Cu at (183.5, 51.0)
- added R5: 8.2k, Resistor_SMD:R_0805_2012Metric_Pad1.20x1.40mm_HandSolder, F.Cu at (193.5, 51.0)
- added R6: 8.2k, Resistor_SMD:R_0805_2012Metric_Pad1.20x1.40mm_HandSolder, F.Cu at (179.5, 45.5)
- added R7: 8.2k, Resistor_SMD:R_0805_2012Metric_Pad1.20x1.40mm_HandSolder, F.Cu at (177.0, 54.5)
- added R8: 8.2k, Resistor_SMD:R_0805_2012Metric_Pad1.20x1.40mm_HandSolder, F.Cu at (168.5, 45.5)
- added R9: 8.2k, Resistor_SMD:R_0805_2012Metric_Pad1.20x1.40mm_HandSolder, F.Cu at (213.0, 39.5)
- added RESET1: SW_Push, LCSC:SW-SMD_4P-L4.2-W3.2-P2.15-LS4.6, F.Cu at (156.5, 47.5)
- added WAKE1: SW_Push, LCSC:SW-SMD_4P-L4.2-W3.2-P2.15-LS4.6, F.Cu at (152.8, 51.8)
Connections:
- U1 pad 1: unconnected-(U1-RESET-Pad1) -> RESET
Routing:
- net +3.3V: track 59.4 -> 78.4 mm, vias 1 -> 4
- net Net-(R11-Pad1): track 0.00 -> 11.2 mm
- net COL7: track 169.6 -> 159.5 mm
- net RESET: track 0.00 -> 8.20 mm
- net COL8: track 159.0 -> 167.0 mm, vias 15 -> 17
- net COL3: track 151.8 -> 154.1 mm, vias 7 -> 10
- net CMD: track 96.3 -> 97.2 mm
- net ROW9: track 77.1 -> 77.9 mm
- net GND: track 49.3 -> 49.6 mm, vias 1 -> 70
- net COL1: track 132.8 -> 132.9 mm, vias 17 -> 19
- added copper zone on B.Cu, net GND
- added copper zone on F.Cu, net GND
Other:
- outline, holes or cut-outs redrawn
- board text added: "4"
- board text added: "R"
- board text added: "RESET"
- board text added: "WAKE"
- board text removed: "CMD"
- board text removed: "COL1"
- board text removed: "COL8"
- board text removed: "ROW1"
- board text removed: "ROW7"
- board text removed: "ROW9"
