File: KanaType.kicad_sch (KiCad schematic)
At the start: 61 parts, among them J1 Conn_01x04_Socket, SW1 SW_Push, SW10 SW_Push, SW11 SW_Push, SW12 SW_Push, SW13 SW_Push, SW14 SW_Push, SW15 SW_Push, SW16 SW_Push, SW17 SW_Push, SW18 SW_Push, SW19 SW_Push, SW2 SW_Push, SW20 SW_Push, SW21 SW_Push, SW22 SW_Push, SW23 SW_Push, SW24 SW_Push, SW25 SW_Push, SW26 SW_Push, SW27 SW_Push, SW28 SW_Push, SW29 SW_Push, SW3 SW_Push, SW30 SW_Push, SW31 SW_Push, SW32 SW_Push, SW33 SW_Push, SW34 SW_Push, SW35 SW_Push, SW36 SW_Push, SW37 SW_Push, SW38 SW_Push, SW39 SW_Push, SW4 SW_Push, SW40 SW_Push, SW41 SW_Push, SW42 SW_Push, SW43 SW_Push, SW44 SW_Push, SW45 SW_Push, SW46 SW_Push, SW47 SW_Push, SW48 SW_Push, SW49 SW_Push, SW5 SW_Push, SW51 SW_Push, SW53 SW_Push, SW55 SW_Push, SW57 SW_Push, SW59 SW_Push, SW6 SW_Push, SW61 SW_Push, SW63 SW_Push, SW7 SW_Push, SW8 SW_Push, SW9 SW_Push, U1 Adafruit-Feather-RP2040

Commit message: Main Version
Connections:
- net ROW1: no longer SW1.3, SW2.3, SW3.3, SW4.3, SW5.3, SW6.3, SW7.3, SW8.3
- net ROW2: no longer SW10.3, SW11.3, SW12.3, SW13.3, SW14.3, SW15.3, SW16.3, SW9.3
- net ROW3: no longer SW17.3, SW19.3, SW21.3, SW23.3, SW25.3, SW27.3, SW29.3, SW31.3
- net ROW4: no longer SW18.3, SW20.3, SW22.3, SW24.3, SW26.3, SW28.3, SW30.3, SW32.3
- net ROW5: no longer SW33.3, SW35.3, SW37.3, SW39.3, SW41.3, SW43.3, SW45.3, SW47.3
- net ROW6: no longer SW34.3, SW36.3, SW38.3, SW40.3, SW42.3, SW44.3, SW46.3, SW48.3
- net ROW7: no longer SW49.3, SW51.3, SW53.3, SW55.3, SW57.3, SW59.3, SW61.3, SW63.3
Other:
- moved on the sheet: J1
